Commit message: Replaced ur10 collision models with primitive shapes

File: ur_description/urdf/ur10.urdf.xacro (robot description, xacro)
@@ -71,6 +71,7 @@
       <collision>
         <geometry>
-          <mesh filename="package://ur_description/meshes/ur10/collision/base.stl"/>
-        </geometry>
+          <box size="0.3 0.4 1.4"/>
+        </geometry>
+        <origin xyz="0 0 -0.7"/>
       </collision>
       <xacro:cylinder_inertial radius="0.075" length="0.038" mass="${base_mass}">
@@ -102,6 +103,13 @@
       <collision>
         <geometry>
-          <mesh filename="package://ur_description/meshes/ur10/collision/shoulder.stl"/>
-        </geometry>
+          <cylinder length="0.215" radius="0.08"/>
+        </geometry>
+        <origin xyz="0 0 -0.0175"/>
+      </collision>
+      <collision>
+        <geometry>
+          <cylinder length="0.265" radius="0.08"/>
+        </geometry>
+        <origin xyz="0 0.1325 0" rpy="${pi/2} 0 0"/>
       </collision>
       <xacro:cylinder_inertial radius="0.075" length="0.178" mass="${shoulder_mass}">
@@ -133,6 +141,13 @@
       <collision>
         <geometry>
-          <mesh filename="package://ur_description/meshes/ur10/collision/upperarm.stl"/>
-        </geometry>
+          <cylinder length="0.527" radius="0.06"/>
+        </geometry>
+        <origin xyz="0 -0.045 0.35"/>
+      </collision>
+      <collision>
+        <geometry>
+          <cylinder length="0.27" radius="0.063"/>
+        </geometry>
+        <origin xyz="0 -0.11 0.612" rpy="${pi/2} 0 0"/>
       </collision>
       <xacro:cylinder_inertial radius="0.075" length="${-ur10_a2}" mass="${upper_arm_mass}">
@@ -164,6 +179,13 @@
       <collision>
         <geometry>
-          <mesh filename="package://ur_description/meshes/ur10/collision/forearm.stl"/>
-        </geometry>
+          <cylinder length="0.5" radius="0.05"/>
+        </geometry>
+        <origin xyz="0 0 0.32"/>
+      </collision>
+      <collision>
+        <geometry>
+          <cylinder length="0.12" radius="0.05"/>
+        </geometry>
+        <origin xyz="0 0 0.57" rpy="${pi/2} 0 0"/>
       </collision>
       <xacro:cylinder_inertial radius="0.075" length="${-ur10_a3}" mass="${forearm_mass}">
@@ -193,9 +215,4 @@
         </material>
       </visual>
-      <collision>
-        <geometry>
-          <mesh filename="package://ur_description/meshes/ur10/collision/wrist1.stl"/>
-        </geometry>
-      </collision>
       <xacro:cylinder_inertial radius="0.075" length="0.12" mass="${wrist_1_mass}">
         <origin xyz="0.0 0.0 0.0" rpy="0 0 0" />
@@ -226,6 +243,13 @@
       <collision>
         <geometry>
-          <mesh filename="package://ur_description/meshes/ur10/collision/wrist2.stl"/>
-        </geometry>
+          <cylinder length="0.18" radius="0.05"/>
+        </geometry>
+        <origin xyz="0 0 0.03"/>
+      </collision>
+      <collision>
+        <geometry>
+          <cylinder length="0.155" radius="0.05"/>
+        </geometry>
+        <origin xyz="0 0.0175 0.12" rpy="${pi/2} 0 0"/>
       </collision>
       <xacro:cylinder_inertial radius="0.075" length="0.12" mass="${wrist_2_mass}">
@@ -270,10 +294,4 @@
     </joint>
     <link name="${prefix}ee_link">
-      <collision>
-        <geometry>
-          <box size="0.01 0.01 0.01"/>
-        </geometry>
-        <origin rpy="0 0 0" xyz="-0.01 0 0"/>
-      </collision>
     </link>
     <xacro:ur_arm_transmission prefix="${prefix}" />

Commit message: cleanup: Removed obsolete collision models

File: ur_description/urdf/ur10.urdf.xacro (robot description, xacro)
@@ -69,10 +69,4 @@
         </material>
       </visual>
-      <collision>
-        <geometry>
-          <box size="0.3 0.4 1.4"/>
-        </geometry>
-        <origin xyz="0 0 -0.7"/>
-      </collision>
       <xacro:cylinder_inertial radius="0.075" length="0.038" mass="${base_mass}">
         <origin xyz="0.0 0.0 0.0" rpy="0 0 0" />
@@ -279,9 +273,4 @@
         </material>
       </visual>
-      <collision>
-        <geometry>
-          <mesh filename="package://ur_description/meshes/ur10/collision/wrist3.stl"/>
-        </geometry>
-      </collision>
       <xacro:cylinder_inertial radius="0.075" length="0.12" mass="${wrist_3_mass}">
         <origin xyz="0.0 0.0 0.0" rpy="0 0 0" />

Commit message: update(ur10): added collision ignores

File: ur_description/urdf/ur10.urdf.xacro (robot description, xacro)
@@ -143,5 +143,5 @@
           <cylinder length="0.27" radius="0.063"/>
         </geometry>
-        <origin xyz="0 -0.11 0.612" rpy="${pi/2} 0 0"/>
+        <origin xyz="0 -0.11 ${upper_arm_length}" rpy="${pi/2} 0 0"/>
       </collision>
       <xacro:cylinder_inertial radius="0.075" length="${-ur10_a2}" mass="${upper_arm_mass}">
@@ -179,7 +179,7 @@
       <collision>
         <geometry>
-          <cylinder length="0.12" radius="0.05"/>
-        </geometry>
-        <origin xyz="0 0 0.57" rpy="${pi/2} 0 0"/>
+          <cylinder length="0.17" radius="0.05"/>
+        </geometry>
+        <origin xyz="0 0.025 ${forearm_length}" rpy="${pi/2} 0 0"/>
       </collision>
       <xacro:cylinder_inertial radius="0.075" length="${-ur10_a3}" mass="${forearm_mass}">
@@ -241,10 +241,4 @@
         <origin xyz="0 0 0.03"/>
       </collision>
-      <collision>
-        <geometry>
-          <cylinder length="0.155" radius="0.05"/>
-        </geometry>
-        <origin xyz="0 0.0175 0.12" rpy="${pi/2} 0 0"/>
-      </collision>
       <xacro:cylinder_inertial radius="0.075" length="0.12" mass="${wrist_2_mass}">
         <origin xyz="0.0 0.0 0.0" rpy="0 0 0" />
@@ -273,4 +267,10 @@
         </material>
       </visual>
+      <collision>
+        <geometry>
+          <cylinder length="0.155" radius="0.05"/>
+        </geometry>
+        <origin xyz="0 0.0175 0" rpy="${pi/2} 0 0"/>
+      </collision>
       <xacro:cylinder_inertial radius="0.075" length="0.12" mass="${wrist_3_mass}">
         <origin xyz="0.0 0.0 0.0" rpy="0 0 0" />
@@ -304,4 +304,8 @@
       <child link="${prefix}tool0"/>
     </joint>
+    <sr_ignore_collisions link1="${prefix}shoulder_link" link2="${prefix}upper_arm_link"/>
+    <sr_ignore_collisions link1="${prefix}upper_arm_link" link2="${prefix}forearm_link"/>
+    <sr_ignore_collisions link1="${prefix}forearm_link" link2="${prefix}wrist_2_link"/>
+    <sr_ignore_collisions link1="${prefix}wrist_2_link" link2="${prefix}wrist_3_link"/>
   </xacro:macro>
 </robot>

Commit message: fix: removed pi property from ur description files.

File: ur_description/urdf/ur10.urdf.xacro (robot description, xacro)
@@ -7,5 +7,4 @@
   <xacro:include filename="$(find ur_description)/urdf/ur.transmission.xacro" />
   <xacro:include filename="$(find ur_description)/urdf/ur.gazebo.xacro" />
-  <xacro:property name="pi" value="3.14159265" />
   <!-- Inertia parameters -->
   <xacro:property name="base_mass" value="4.0" />  <!-- This mass might be incorrect -->

Commit message: removed all visual geometry except for wrists

File: ur_description/urdf/ur10.urdf.xacro (robot description, xacro)
@@ -60,5 +60,5 @@
 		 wrist_3_lower_limit:=${-pi}    wrist_3_upper_limit:=${pi}">
     <link name="${prefix}base_link" >
-      <visual>
+      <!-- <visual>
         <geometry>
           <mesh filename="package://ur_description/meshes/ur10/visual/base.dae"/>
@@ -67,5 +67,5 @@
           <color rgba="0.7 0.7 0.7 1.0"/>
         </material>
-      </visual>
+      </visual> -->
       <xacro:cylinder_inertial radius="0.075" length="0.038" mass="${base_mass}">
         <origin xyz="0.0 0.0 0.0" rpy="0 0 0" />
@@ -86,5 +86,5 @@
     </joint>
     <link name="${prefix}shoulder_link">
-      <visual>
+<!--       <visual>
         <geometry>
           <mesh filename="package://ur_description/meshes/ur10/visual/shoulder.dae"/>
@@ -93,5 +93,5 @@
           <color rgba="0.7 0.7 0.7 1.0"/>
         </material>
-      </visual>
+      </visual> -->
       <collision>
         <geometry>
@@ -124,5 +124,5 @@
     </joint>
     <link name="${prefix}upper_arm_link">
-      <visual>
+<!--       <visual>
         <geometry>
           <mesh filename="package://ur_description/meshes/ur10/visual/upperarm.dae"/>
@@ -131,5 +131,5 @@
           <color rgba="0.7 0.7 0.7 1.0"/>
         </material>
-      </visual>
+      </visual> -->
       <collision>
         <geometry>
@@ -162,5 +162,5 @@
     </joint>
     <link name="${prefix}forearm_link">
-      <visual>
+<!--       <visual>
          <geometry>
           <mesh filename="package://ur_description/meshes/ur10/visual/forearm.dae"/>
@@ -169,5 +169,5 @@
           <color rgba="0.7 0.7 0.7 1.0"/>
         </material>
-      </visual>
+      </visual> -->
       <collision>
         <geometry>
